File: KiCad/OLED.kicad_pcb (KiCad board)
At the start: 2 copper layers, 44.5 x 37 mm, 17 parts, among them J1 USB-C, J2 DC, J3 GPIO, M1 D24V5F3-NoSHDN, M2 OLED1.5-RGB, M3 SCD30-4pin, U1 FT230XQ, U2 ESP32-WROOM-32

Commit message: Tracked
Parts:
- added REF**: AJK, RevK:AJK, B.Cu at (130.8, 87.0)
- added REF**: AJK, RevK:AJK, F.Cu at (134.8, 89.5)
- J2: moved to F.Cu
- turned J2 to 90 degrees
Connections:
- J3 pad 2: Net-(J3-Pad2) -> IO1
- J3 pad 3: Net-(J3-Pad3) -> IO2
- J3 pad 4: Net-(J3-Pad4) -> IO3
- J3 pad 5: Net-(J3-Pad5) -> IO4
- J3 pad 6: Net-(J3-Pad6) -> IO5
- J3 pad 7: Net-(J3-Pad7) -> IO6
- J3 pad 8: Net-(J3-Pad8) -> IO7
- M2 pad 3: Net-(M2-Pad3) -> OLED-MOSI
- M2 pad 4: Net-(M2-Pad4) -> OLED-SCLK
- M2 pad 5: Net-(M2-Pad5) -> OLED-CS0
- M2 pad 6: Net-(M2-Pad6) -> OLED-DC
- M2 pad 7: Net-(M2-Pad7) -> OLED-RST
- M3 pad 3: Net-(M3-Pad3) -> CO2-SCL
- M3 pad 4: Net-(M3-Pad4) -> CO2-SDA
- R3 pad 1: Net-(J3-Pad2) -> IO1
- R4 pad 1: Net-(J3-Pad3) -> IO2
- R5 pad 1: Net-(J3-Pad4) -> IO3
- R6 pad 1: Net-(J3-Pad5) -> IO4
- R7 pad 1: Net-(J3-Pad6) -> IO5
- R8 pad 1: Net-(J3-Pad7) -> IO6
- R9 pad 1: Net-(J3-Pad8) -> IO7
- U1 pad 8: Net-(U1-Pad8) -> +3V3
- U1 pad 9: Net-(U1-Pad8) -> +3V3
- U2 pad 11: Net-(U2-Pad11) -> OLED-DC
- U2 pad 12: Net-(U2-Pad12) -> OLED-RST
- U2 pad 13: Net-(U2-Pad13) -> OLED-SCLK
- U2 pad 16: Net-(U2-Pad16) -> OLED-MOSI
- U2 pad 23: Net-(U2-Pad23) -> OLED-CS0
- U2 pad 26: Net-(U2-Pad26) -> IO1
- U2 pad 27: Net-(U2-Pad27) -> IO2
- U2 pad 28: Net-(U2-Pad28) -> IO3
- U2 pad 29: Net-(U2-Pad29) -> IO4
- U2 pad 30: Net-(U2-Pad30) -> IO5
- U2 pad 31: Net-(U2-Pad31) -> IO6
- U2 pad 33: Net-(U2-Pad33) -> IO7
- U2 pad 34: Net-(U2-Pad34) -> Net-(U1-Pad15)
- U2 pad 35: Net-(U2-Pad35) -> Net-(U1-Pad2)
- U2 pad 6: Net-(U2-Pad6) -> CO2-SDA
- U2 pad 7: Net-(U2-Pad7) -> CO2-SCL
Routing:
- net +3V3: track 0.00 -> 74.7 mm, vias 0 -> 1
- net GND: track 0.00 -> 62.0 mm, vias 0 -> 1
- net Net-(U1-Pad2): track 0.00 -> 47.8 mm, vias 0 -> 2
- net Net-(U1-Pad16): track 0.00 -> 42.5 mm, vias 0 -> 2
- net OLED-CS0: track 0.00 -> 38.5 mm, vias 0 -> 1
- net Net-(U1-Pad15): track 0.00 -> 35.3 mm, vias 0 -> 2
- net IO3: track 0.00 -> 30.8 mm
- net Net-(J1-PadA4): track 0.00 -> 29.8 mm
- net OLED-MOSI: track 0.00 -> 27.6 mm, vias 0 -> 1
- net Net-(U1-Pad14): track 0.00 -> 27.5 mm, vias 0 -> 2
- net OLED-SCLK: track 0.00 -> 23.8 mm, vias 0 -> 1
- net OLED-RST: track 0.00 -> 23.7 mm, vias 0 -> 1
- net IO7: track 0.00 -> 21.9 mm
- net OLED-DC: track 0.00 -> 20.8 mm, vias 0 -> 1
- net IO2: track 0.00 -> 19.8 mm
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Other:
- board text added: "www.me.uk"
